Commit message: fast_lio

File: rigel_description/urdf/rigel.urdf.xacro (robot description, xacro)
@@ -1,10 +1,12 @@
 <?xml version="1.0"?>
-<robot name="scout_mini"
+<robot name="rigel"
     xmlns:xacro="http://ros.org/wiki/xacro">
-    <xacro:property name="M_PI" value="3.141592653" />
-    <xacro:include filename="$(find scout_description)/urdf/scout_mini.xacro" />
+    <xacro:property name="PI" value="3.141592653" />
+    <xacro:property name="rail_top_offset" value="0.069" />
+    <xacro:property name="rail_front_offset" value="0.175" />
+    <xacro:include filename="$(find scout_description)/urdf/scout_mini.urdf.xacro" />
     <xacro:include filename="$(find rigel_description)/urdf/slam_sys.urdf.xacro"/>
     <xacro:ice9_slam parent="base_link" name="slamsys">
-        <origin xyz="0 0.161438 ${0.335382 + wheel_radius}" rpy="0 0 0" />
+        <origin xyz="${-0.002 + rail_front_offset} 0 ${0.17 + rail_top_offset}" rpy="0 0 ${-PI/2}" />
     </xacro:ice9_slam>
 </robot>

File: rigel_description/urdf/slam_sys.urdf.xacro (robot description, xacro)
@@ -1,4 +1,4 @@
 <?xml version="1.0"?>
-<robot xmlns:xacro="http://www.ros.org/wiki/xacro" name="LSC16">
+<robot xmlns:xacro="http://www.ros.org/wiki/xacro" name="slam_sys">
     <xacro:macro name="ice9_slam" params="*origin parent:=base_link name:=slam_sys">
         <joint name="${name}_base_mount_joint" type="fixed">
@@ -20,15 +20,28 @@
         </link>
         <xacro:include filename="$(find velodyne_description)/urdf/VLP-16.urdf.xacro" />
-    <xacro:VLP-16 parent="${name}_base_link" name="velodyne">
-        <origin xyz="0 0 0" rpy="0 0 -${M_PI/2}" />
-    </xacro:VLP-16>
+        <xacro:VLP-16 parent="${name}_base_link" name="velodyne">
+            <origin xyz="0 0 0" rpy="0 0 -${M_PI/2}" />
+        </xacro:VLP-16>
         <xacro:include filename="$(find realsense2_description)/urdf/_d435i.urdf.xacro" />
-    <xacro:sensor_d435i parent="${name}_base_link" name="realsense">
-        <origin xyz="0 0.06185 -0.0495" rpy="0 0 ${M_PI/2}" />
-    </xacro:sensor_d435i>
+        <xacro:sensor_d435i parent="${name}_base_link" name="realsense">
+            <origin xyz="0 0.06185 -0.0495" rpy="0 0 ${M_PI/2}" />
+        </xacro:sensor_d435i>
         <xacro:include filename="$(find lslidar_description)/urdf/LSC16.urdf.xacro" />
         <xacro:LSC16 parent="${name}_base_link" name="lslidar">
             <origin xyz="0 -0.055 -0.070" rpy="-${M_PI/2} 0 ${M_PI}" />
         </xacro:LSC16>
+        <link name="microstrain_link">
+            <visual>
+                <geometry>
+                    <box size="0.0244 0.0232 0.015" />
+                </geometry>
+            </visual>
+        </link>
+        <joint name="{name}_microstrain_link_joint" type="fixed">
+            <!-- <origin xyz="-0.0917 -0.00485 -0.1365" rpy="0 0 0" /> -->
+            <origin xyz="0.0917 ${- 0.0329/2 + 0.0213} ${-0.140 + 0.0075}" rpy="${M_PI} 0 ${-M_PI/2}" />
+            <parent link="${name}_base_link" />
+            <child link="microstrain_link" />
+        </joint>
     </xacro:macro>
 </robot>
